File: BLOCKSmodular-hardware.kicad_pcb (KiCad board)
At the start: 2 copper layers, 96 x 95 mm, 75 parts, among them J1 THONKICONN, J10 Bela_AudioOut, J11 THONKICONN, J12 THONKICONN, J13 THONKICONN, J14 THONKICONN, J15 Bela_P9, J16 Bela_P8, J17 EurorackPower, J18 THONKICONN, J19 THONKICONN, J2 THONKICONN, J3 THONKICONN, J4 Bela_AnalogOut, J5 THONKICONN, J6 THONKICONN, J7 THONKICONN, J8 THONKICONN, J9 THONKICONN, SW1 NKK_NR01, U1 TL074, U2 TL074, U3 ADA4075-2, U4 TL074

Commit message: Update: 基板修正
Parts:
- moved C14 9.50 mm to (114.7, 41.8), turned to 270 degrees
- moved C9 7.24 mm to (92.8, 28.8), turned to 180 degrees
- moved C10 6.79 mm to (89.2, 33.9), turned to 90 degrees
- moved C12 2.62 mm to (103.2, 45.7), turned to 90 degrees
- moved R16 0.72 mm to (109.4, 53.2)
- moved R15 0.72 mm to (107.2, 53.1)
- moved R10 0.58 mm to (109.5, 58.0)
- moved R9 0.58 mm to (107.2, 57.9)
- moved C3 0.38 mm to (112.7, 59.4)
- moved C5 0.37 mm to (96.9, 66.2)
- moved G*** 0.31 mm to (147.0, 41.5)
- moved R1 0.25 mm to (107.5, 74.5)
- moved R2 0.22 mm to (109.8, 74.6)
- renumbered R20 to R19, R19 to R20, R24 to R23, R23 to R24, R27 to R25, R28 to R26, R25 to R27, R26 to R28
Connections:
- C5 pad 2: -12V -> +12V
- C6 pad 2: +12V -> -12V
- J15 pad 11: (no net) -> Net-(J15-Pad11)
- J15 pad 12: Net-(J15-Pad12) -> (no net)
- J15 pad 13: (no net) -> Net-(J15-Pad13)
- J15 pad 14: Net-(J15-Pad14) -> (no net)
- J15 pad 15: (no net) -> Net-(J15-Pad15)
- J15 pad 16: Net-(J15-Pad16) -> (no net)
- J15 pad 5: (no net) -> +5V
- J15 pad 6: +5V -> (no net)
- R19 pad 1: Net-(R19-Pad2) -> Net-(R19-Pad1)
- R19 pad 2: Net-(J10-Pad2) -> GND
- R20 pad 2: Net-(R19-Pad2) -> Net-(R19-Pad1)
- R23 pad 2: Net-(J15-Pad12) -> Net-(J15-Pad11)
- R25 pad 2: Net-(J15-Pad14) -> Net-(J15-Pad13)
- R26 pad 2: Net-(J15-Pad16) -> Net-(J15-Pad15)
- SW1 pad 2: Net-(J15-Pad12) -> Net-(J15-Pad11)
- SW1 pad 4: Net-(J15-Pad14) -> Net-(J15-Pad13)
- SW1 pad 6: Net-(J15-Pad16) -> Net-(J15-Pad15)
- U3 pad 4: +12V -> -12V
- U3 pad 5: Net-(R19-Pad2) -> Net-(J10-Pad2)
- U3 pad 6: GND -> Net-(R19-Pad1)
- U3 pad 8: -12V -> +12V
Routing:
- net GND: track 188.5 -> 119.5 mm, vias 39 -> 32
- net Net-(J15-Pad15): track 0.00 -> 28.1 mm
- net Net-(J15-Pad16): track 24.6 -> 0.00 mm
- net Net-(J15-Pad13): track 0.00 -> 21.4 mm
- net Net-(J15-Pad14): track 18.1 -> 0.00 mm
- net Net-(J7-Pad3): track 76.9 -> 61.4 mm, vias 2 -> 0
- net Net-(J15-Pad11): track 0.00 -> 15.2 mm
- net Net-(J15-Pad12): track 12.7 -> 0.00 mm
- net -12V: track 145.1 -> 134.9 mm, vias 4 -> 2
- net Net-(R19-Pad1): track 0.00 -> 5.85 mm
- net +12V: track 151.2 -> 146.2 mm, vias 4 -> 5
- net Net-(R19-Pad2): track 4.71 -> 0.00 mm
- net Net-(J10-Pad2): track 62.5 -> 66.9 mm
- net +5V: track 40.2 -> 36.6 mm, vias 1 -> 0
- net Net-(J3-Pad3): track 54.7 -> 52.0 mm
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Other:
- board text added: "Audio Out"
- board text added: "CV Out"
- board text added: "Gate Out"
- board text added: "Lch"
- board text added: "Rch"
- board text removed: "Audio Lch"
- board text removed: "Audio Rch"
